Commit message: It is working but need some adjustments

File: sim_ws/src/Simulations/blender_gazebo/sdf/landmark.sdf.xacro (robot description, xacro)
@@ -3,9 +3,9 @@
   <xacro:macro name="landmark" params="id *pose">
     <xacro:property name="pole_above_ground" value="0.3"/>
-    <xacro:property name="box_width" value="0.25"/>
+    <xacro:property name="box_width" value="0.20"/>
     <xacro:property name="pole_below_ground" value="0.1"/>
     <xacro:property name="box_height" value="0.32"/>
     <xacro:property name="sheet_width" value="0.005"/> <!-- When the sheet is too thin it is not shaded properly for some reason -->
-    <xacro:property name="sheet_out" value="0.001"/>
+    <xacro:property name="sheet_out" value="0.01"/>
     <model name="landmark${id}">
       <xacro:insert_block name="pose"/>
@@ -36,9 +36,10 @@
         </collision>
         <visual name="box_visual">
-          <pose>0 0 ${pole_above_ground + box_height/2} 0 0 0</pose>
+          <pose>0 0 ${-0.15+pole_above_ground + box_height/2} 0 0 +${pi/3}</pose>
           <geometry>
-            <box>
-              <size>${box_width} ${box_width} ${box_height}</size>
-            </box>
+            <mesh>
+              <uri>/home/halil/Documents/sim_ws/src/Simulations/blender_gazebo/sdf/meshes/ERC_Sign.stl</uri> <!-- Change dictionary line-->
+              <scale>0.0013 0.0013 0.001</scale>
+            </mesh>
           </geometry>
           <material>
@@ -49,9 +50,10 @@
         </visual>
         <collision name="box_collision">
-          <pose>0 0 ${pole_above_ground + box_height/2} 0 0 0</pose>
+          <pose>0 0 ${-0.15+pole_above_ground + box_height/2} 0 0 +${pi/3}</pose>
           <geometry>
-            <box>
-              <size>${box_width} ${box_width} ${box_height}</size>
-            </box>
+            <mesh>
+              <uri>/home/halil/Documents/sim_ws/src/Simulations/blender_gazebo/sdf/meshes/ERC_Sign.stl</uri> <!-- Change dictionary line-->
+              <scale>0.0013 0.0013 0.001</scale>
+            </mesh>
           </geometry>
         </collision>
@@ -72,14 +74,14 @@
         </xacro:macro>
         <xacro:landmark_sheet name="sheet1">
-          <pose>0 ${(box_width - sheet_width)/2 + sheet_out} ${pole_above_ground + box_height/2} 0 0 0</pose>
+          <pose>0 ${(box_width - sheet_width)/2} ${pole_above_ground + box_height/2} 0 0 0</pose>
         </xacro:landmark_sheet>
-        <xacro:landmark_sheet name="sheet2">
+        <!-- <xacro:landmark_sheet name="sheet2">
           <pose>0 -${(box_width - sheet_width)/2 + sheet_out} ${pole_above_ground + box_height/2} 0 0 0</pose>
-        </xacro:landmark_sheet>
+        </xacro:landmark_sheet> -->
         <xacro:landmark_sheet name="sheet3">
-          <pose>${(box_width - sheet_width)/2 + sheet_out} 0 ${pole_above_ground + box_height/2} 0 0 ${pi/2}</pose>
+          <pose>${((box_width-0.05) - sheet_width)/2 + sheet_out} -0.06 ${pole_above_ground + box_height/2} 0 0 +${pi/3}</pose>
         </xacro:landmark_sheet>
         <xacro:landmark_sheet name="sheet4">
-          <pose>-${(box_width - sheet_width)/2 + sheet_out} 0 ${pole_above_ground + box_height/2} 0 0 ${pi/2}</pose>
+          <pose>-${((box_width-0.06) - sheet_width)/2 + sheet_out} -0.06 ${pole_above_ground + box_height/2} 0 0 -${pi/3}</pose>
         </xacro:landmark_sheet>
       </link>

File: sim_ws/src/Simulations/blender_gazebo/worlds/marsyard2021.world.xacro (robot description, xacro)
@@ -1,5 +1,9 @@
 <?xml version="1.0"?>
-<sdf version="1.6" xmlns:xacro="http://www.ros.org/wiki/xacro">
+<sdf version="1.6"
+  xmlns:xacro="http://www.ros.org/wiki/xacro">
   <world name="marsyard2021">
+<!--
+@author: Baran Berk Bağcı-->
+<!-- Empty world with artag, blue sky and clouds.-->
     <physics type="ode">
       <ode>
@@ -25,48 +29,92 @@
       </sky>
       <shadows>true</shadows>
-      <origin_visual>false</origin_visual>
+      <origin_visual>true</origin_visual>
     </scene>
+    <include>
+      <uri>model://ground_plane</uri>
+    </include>
+    <!-- Actors is model with automated moving models in gazebo in this cas our actor is cosmonaut named Lagari Hasan Çelebi.-->
+    <actor name="Lâgari Hasan Çelebi">
+      <link name="cosmonaut">
+        <visual name="visual">
+          <pose>0 25 0.9 0 0 1.57</pose>
+          <geometry>
+            <mesh>
+              <scale>1 1 1</scale>
+              <uri>/home/baran/rover_simulation_ws/src/Simulations/blender_gazebo/worlds/cosmonaut-dae/cosmonaut.dae</uri> <!-- Change this path if you want cosmounaut you can use pwd command on terminal.-->
+            </mesh>
+          </geometry>
+        </visual>
+      </link>
+      <script>
+        <loop>true</loop>
+        <auto_start>true</auto_start>
+        <trajectory id="0" type="square">
+          <waypoint>
+            <time>0.0</time>
+            <pose>-1 -1 0 0 0 0</pose>
+          </waypoint>
+          <waypoint>
+            <time>30.0</time>
+            <pose>20 -1 0 0 0 0</pose>
+          </waypoint>
+          <!-- <waypoint>
+            <time>2.0</time>
+            <pose>1 1 1 0 0 0</pose>
+          </waypoint>
+          <waypoint>
+            <time>3.0</time>
+            <pose>1 -1 1 0 0 0</pose>
+          </waypoint>
+          <waypoint>
+            <time>4.0</time>
+            <pose>-1 -1 1 0 0 0</pose>
+          </waypoint> -->
+        </trajectory>
+      </script>
+    </actor>
     <xacro:include filename="$(find blender_gazebo)/sdf/landmark.sdf.xacro"/>
+    <!-- Artag ids from 1 to 15-->
     <xacro:landmark id="1">
-      <pose>-2.60 -5.17 1.42 0 0 0</pose>
+      <pose>-2.60 -5.17 0.42 0 0 0</pose>
     </xacro:landmark>
     <xacro:landmark id="2">
-      <pose>-6.05 -5.75 1.22 0 0 1.33</pose>
+      <pose>-6.05 -5.75 0.22 0 0 1.33</pose>
     </xacro:landmark>
     <xacro:landmark id="3">
-      <pose>-7.93 18.45 1.21 0 0 0.35</pose>
+      <pose>-7.93 18.45 0.21 0 0 0.35</pose>
     </xacro:landmark>
     <xacro:landmark id="4">
-      <pose>-0.23 9.19 1.29 0 0 0.98</pose>
+      <pose>-0.23 9.19 0.29 0 0 0.98</pose>
     </xacro:landmark>
     <xacro:landmark id="5">
-      <pose>-12.3 -6.28 1.16 0 0 1.47</pose>
+      <pose>-12.3 -6.28 0.16 0 0 1.47</pose>
     </xacro:landmark>
     <xacro:landmark id="6">
-      <pose>18.46 -1.15 1.28 0 0 0.83</pose>
+      <pose>18.46 -1.15 0.28 0 0 0.83</pose>
     </xacro:landmark>
     <xacro:landmark id="7">
-      <pose>13.07 -7.09 1.32 0 0 1.19</pose>
+      <pose>13.07 -7.09 0.32 0 0 1.19</pose>
     </xacro:landmark>
     <xacro:landmark id="8">
-      <pose>3.05 17.20 1.19 0 0 0.95</pose>
+      <pose>3.05 17.20 0.19 0 0 0.95</pose>
     </xacro:landmark>
     <xacro:landmark id="9">
-      <pose>-14.82 1.52 1.20 0 0 0.16</pose>
+      <pose>-14.82 1.52 0.20 0 0 0.16</pose>
     </xacro:landmark>
     <xacro:landmark id="10">
-      <pose>-10.74 -15.05 1.29 0 0 1.27</pose>
+      <pose>-10.74 -15.05 0.29 0 0 1.27</pose>
     </xacro:landmark>
     <xacro:landmark id="11">
-      <pose>18.43 5.48 1.36 0 0 0.23</pose>
+      <pose>18.43 5.48 0.36 0 0 0.23</pose>
     </xacro:landmark>
     <xacro:landmark id="12">
-      <pose>-4.14 4.51 1.12 0 0 0.47</pose>
+      <pose>-4.14 4.51 0.12 0 0 0.47</pose>
     </xacro:landmark>
     <xacro:landmark id="13">
-      <pose>9.78 5.39 1.35 0 0 1.13</pose>
+      <pose>9.78 5.39 0.35 0 0 1.13</pose>
     </xacro:landmark>
     <xacro:landmark id="15">
-      <pose>15.60 -9.14 1.15 0 0 1.20</pose>
+      <pose>15.60 -9.14 0.15 0 0 1.20</pose>
     </xacro:landmark>
   </world>

Commit message: Working_state_machine

File: sim_ws/src/Simulations/blender_gazebo/sdf/landmark.sdf.xacro (robot description, xacro)
@@ -1,4 +1,6 @@
 <?xml version="1.0"?>
 <sdf version="1.6" xmlns:xacro="http://www.ros.org/wiki/xacro">
+<!--
+@author: Baran Berk Bağcı-->
   <xacro:macro name="landmark" params="id *pose">
     <xacro:property name="pole_above_ground" value="0.3"/>
@@ -35,4 +37,5 @@
           </geometry>
         </collision>
+        <!-- Sign Prism Head-->
         <visual name="box_visual">
           <pose>0 0 ${-0.15+pole_above_ground + box_height/2} 0 0 +${pi/3}</pose>
@@ -45,5 +48,5 @@
           <material>
             <script>
-              <name>ERC_Landmark/Box</name>
+              <name>Gazebo/White</name>
             </script>
           </material>
@@ -59,9 +62,9 @@
         </collision>
         <xacro:macro name="landmark_sheet" params="name *pose">
-          <visual name="${name}">
+          <visual nam e="${name}">
             <xacro:insert_block name="pose"/>
             <geometry>
               <box>
-                <size>0.21 ${sheet_width} 0.297</size>
+                <size>0.22 ${sheet_width} 0.22</size>
               </box>
             </geometry>
@@ -73,13 +76,17 @@
           </visual>
         </xacro:macro>
+        <!-- Artag 1-->
         <xacro:landmark_sheet name="sheet1">
           <pose>0 ${(box_width - sheet_width)/2} ${pole_above_ground + box_height/2} 0 0 0</pose>
         </xacro:landmark_sheet>
+        <!-- Don'T delete this because Artag 2 needed rectangular prism sign-->
         <!-- <xacro:landmark_sheet name="sheet2">
           <pose>0 -${(box_width - sheet_width)/2 + sheet_out} ${pole_above_ground + box_height/2} 0 0 0</pose>
         </xacro:landmark_sheet> -->
+        <!-- Artag 3-->
         <xacro:landmark_sheet name="sheet3">
           <pose>${((box_width-0.05) - sheet_width)/2 + sheet_out} -0.06 ${pole_above_ground + box_height/2} 0 0 +${pi/3}</pose>
         </xacro:landmark_sheet>
+        <!-- Artag 4-->
         <xacro:landmark_sheet name="sheet4">
           <pose>-${((box_width-0.06) - sheet_width)/2 + sheet_out} -0.06 ${pole_above_ground + box_height/2} 0 0 -${pi/3}</pose>

File: sim_ws/src/Simulations/blender_gazebo/worlds/marsyard2021.world.xacro (robot description, xacro)
@@ -59,16 +59,4 @@
             <pose>20 -1 0 0 0 0</pose>
           </waypoint>
-          <!-- <waypoint>
-            <time>2.0</time>
-            <pose>1 1 1 0 0 0</pose>
-          </waypoint>
-          <waypoint>
-            <time>3.0</time>
-            <pose>1 -1 1 0 0 0</pose>
-          </waypoint>
-          <waypoint>
-            <time>4.0</time>
-            <pose>-1 -1 1 0 0 0</pose>
-          </waypoint> -->
         </trajectory>
       </script>
@@ -77,44 +65,44 @@
     <!-- Artag ids from 1 to 15-->
     <xacro:landmark id="1">
-      <pose>-2.60 -5.17 0.42 0 0 0</pose>
+      <pose>-2.60 -5.17 1.42 0 0 0</pose>
     </xacro:landmark>
     <xacro:landmark id="2">
-      <pose>-6.05 -5.75 0.22 0 0 1.33</pose>
+      <pose>-6.05 -5.75 1.22 0 0 1.33</pose>
     </xacro:landmark>
     <xacro:landmark id="3">
-      <pose>-7.93 18.45 0.21 0 0 0.35</pose>
+      <pose>-7.93 18.45 1.21 0 0 0.35</pose>
     </xacro:landmark>
     <xacro:landmark id="4">
-      <pose>-0.23 9.19 0.29 0 0 0.98</pose>
+      <pose>-0.23 9.19 1.29 0 0 0.98</pose>
     </xacro:landmark>
     <xacro:landmark id="5">
-      <pose>-12.3 -6.28 0.16 0 0 1.47</pose>
+      <pose>-12.3 -6.28 1.16 0 0 1.47</pose>
     </xacro:landmark>
     <xacro:landmark id="6">
-      <pose>18.46 -1.15 0.28 0 0 0.83</pose>
+      <pose>18.46 -1.15 1.28 0 0 0.83</pose>
     </xacro:landmark>
     <xacro:landmark id="7">
-      <pose>13.07 -7.09 0.32 0 0 1.19</pose>
+      <pose>13.07 -7.09 1.32 0 0 1.19</pose>
     </xacro:landmark>
     <xacro:landmark id="8">
-      <pose>3.05 17.20 0.19 0 0 0.95</pose>
+      <pose>3.05 17.20 1.19 0 0 0.95</pose>
     </xacro:landmark>
     <xacro:landmark id="9">
-      <pose>-14.82 1.52 0.20 0 0 0.16</pose>
+      <pose>-14.82 1.52 1.20 0 0 0.16</pose>
     </xacro:landmark>
     <xacro:landmark id="10">
-      <pose>-10.74 -15.05 0.29 0 0 1.27</pose>
+      <pose>-10.74 -15.05 1.29 0 0 1.27</pose>
     </xacro:landmark>
     <xacro:landmark id="11">
-      <pose>18.43 5.48 0.36 0 0 0.23</pose>
+      <pose>18.43 5.48 1.36 0 0 0.23</pose>
     </xacro:landmark>
     <xacro:landmark id="12">
-      <pose>-4.14 4.51 0.12 0 0 0.47</pose>
+      <pose>-4.14 4.51 1.12 0 0 0.47</pose>
     </xacro:landmark>
     <xacro:landmark id="13">
-      <pose>9.78 5.39 0.35 0 0 1.13</pose>
+      <pose>9.78 5.39 1.35 0 0 1.13</pose>
     </xacro:landmark>
     <xacro:landmark id="15">
-      <pose>15.60 -9.14 0.15 0 0 1.20</pose>
+      <pose>15.60 -9.14 1.15 0 0 1.20</pose>
     </xacro:landmark>
   </world>
